Commit message: Added caster wheel support

File: simple_diffbot_description/urdf/diffbot.urdf (robot description, URDF)
Before this commit: robot diffbot, 3 links, 2 joints
Links:
- added link caster; collision sphere radius=0.025; visual sphere radius=0.025
Joints:
- added joint caster_joint: type fixed, parent base_link, child caster, origin xyz=-0.12 0 -0.03

Commit message: Adjusted wheel positions for Gazebo visualization

File: simple_diffbot_description/urdf/diffbot.urdf (robot description, URDF)
Before this commit: robot diffbot, 4 links, 3 joints
Joints:
- joint left_wheel_joint: origin xyz=0 0.12 0 -> xyz=0 0.12 -0.05
- joint right_wheel_joint: origin xyz=0 -0.12 0 -> xyz=0 -0.12 -0.05
